File: boop.kicad_pcb (KiCad board)
At the start: 2 copper layers, 74 x 38 mm, 27 parts, among them J1 5V_IN (+/-), J2 PWR_TO_MB, J3 PWR_FROM_CASE, J4 RST_TO_MB, J5 RST_FROM_CASE, J6 XIAO_LEFT_D0-D6, J7 XIAO_RIGHT_5V-D7, J8 PLED_FROM_MB, J9 PLED_TO_CASE, K1 G6K-2F-Y-TR DC5, K2 G6K-2F-Y-TR DC5, U2 LTV-817S-TA1-D, U3 LTV-817S-TA1-D, U4 LTV-817S-TA1-C

Commit message: Updated readme, added esphome yaml
Parts:
- K1, K2: value G6K-2F-Y-TR DC5 -> G6K-2F-Y-TR DC4.5
Changed lines of the file:
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@@
 		(property ki_fp_filters "R_*")
 		(sheetname "/")
-		(sheetfile "esphome-pc-power-dongle.kicad_sch")
+		(sheetfile "boop.kicad_sch")
 		(units
 			(unit
@@
 			)
 		)
-		(property "Value" "G6K-2F-Y-TR DC5"
+		(property "Value" "G6K-2F-Y-TR DC4.5"
 			(at -0.04 6.3 90)
 			(layer "F.Fab")
@@
 			)
 		)
-		(property "LCSC" "C47190"
+		(property "LCSC" "C397193"
 			(at 0 0 90)
 			(unlocked yes)
@@
 		(property ki_fp_filters "Relay*DPDT*Omron*G6K?2*")
 		(sheetname "/")
-		(sheetfile "esphome-pc-power-dongle.kicad_sch")
+		(sheetfile "boop.kicad_sch")
 		(units
 			(unit
@@
 		(property ki_fp_filters "Connector*:*_1x??_*")
 		(sheetname "/")
-		(sheetfile "esphome-pc-power-dongle.kicad_sch")
+		(sheetfile "boop.kicad_sch")
+		(units
+			(unit
+				(name "A")
+				(pins "1" "2")
+			)
+		)
 		(attr through_hole)
 		(duplicate_pad_numbers_are_jumpers no)
@@
 		(property ki_fp_filters "Connector*:*_1x??_*")
 		(sheetname "/")
-		(sheetfile "esphome-pc-power-dongle.kicad_sch")
+		(sheetfile "boop.kicad_sch")
 		(units
 			(unit
@@
 		(property ki_fp_filters "Connector*:*_1x??_*")
 		(sheetname "/")
-		(sheetfile "esphome-pc-power-dongle.kicad_sch")
+		(sheetfile "boop.kicad_sch")
 		(units
 			(unit
@@
 		(property ki_fp_filters "R_*")
 		(sheetname "/")
-		(sheetfile "esphome-pc-power-dongle.kicad_sch")
+		(sheetfile "boop.kicad_sch")
 		(units
 			(unit
@@
 		(property ki_fp_filters "TO-???* *_Diode_* *SingleDiode* D_*")
 		(sheetname "/")
-		(sheetfile "esphome-pc-power-dongle.kicad_sch")
+		(sheetfile "boop.kicad_sch")
 		(units
 			(unit
@@
 		(property ki_fp_filters "R_*")
 		(sheetname "/")
-		(sheetfile "esphome-pc-power-dongle.kicad_sch")
+		(sheetfile "boop.kicad_sch")
 		(units
 			(unit
@@
 		(property ki_fp_filters "C_*")
 		(sheetname "/")
-		(sheetfile "esphome-pc-power-dongle.kicad_sch")
+		(sheetfile "boop.kicad_sch")
 		(units
 			(unit
@@
 		(property ki_fp_filters "R_*")
 		(sheetname "/")
-		(sheetfile "esphome-pc-power-dongle.kicad_sch")
+		(sheetfile "boop.kicad_sch")
 		(units
 			(unit
@@
 		(property ki_fp_filters "Connector*:*_1x??_*")
 		(sheetname "/")
-		(sheetfile "esphome-pc-power-dongle.kicad_sch")
+		(sheetfile "boop.kicad_sch")
 		(units
 			(unit
@@
 		(property ki_fp_filters "SMDIP*W9.53mm*")
 		(sheetname "/")
-		(sheetfile "esphome-pc-power-dongle.kicad_sch")
+		(sheetfile "boop.kicad_sch")
 		(units
 			(unit
@@
 		(property ki_fp_filters "TO-???* *_Diode_* *SingleDiode* D_*")
 		(sheetname "/")
-		(sheetfile "esphome-pc-power-dongle.kicad_sch")
+		(sheetfile "boop.kicad_sch")
+		(units
+			(unit
+				(name "A")
+				(pins "1" "2")
+			)
+		)
 		(attr smd)
 		(duplicate_pad_numbers_are_jumpers no)
@@
 		(property ki_fp_filters "Connector*:*_1x??_*")
 		(sheetname "/")
-		(sheetfile "esphome-pc-power-dongle.kicad_sch")
+		(sheetfile "boop.kicad_sch")
 		(units
 			(unit
@@
 		(property ki_fp_filters "DIP*W7.62mm*")
 		(sheetname "/")
-		(sheetfile "esphome-pc-power-dongle.kicad_sch")
+		(sheetfile "boop.kicad_sch")
 		(units
 			(unit
@@
 		(property ki_fp_filters "Connector*:*_1x??_*")
 		(sheetname "/")
-		(sheetfile "esphome-pc-power-dongle.kicad_sch")
+		(sheetfile "boop.kicad_sch")
 		(units
 			(unit
@@
 		(property ki_fp_filters "Connector*:*_1x??_*")
 		(sheetname "/")
-		(sheetfile "esphome-pc-power-dongle.kicad_sch")
+		(sheetfile "boop.kicad_sch")
 		(units
 			(unit
@@
 		(property ki_fp_filters "Connector*:*_1x??_*")
 		(sheetname "/")
-		(sheetfile "esphome-pc-power-dongle.kicad_sch")
+		(sheetfile "boop.kicad_sch")
 		(units
 			(unit
@@
 		(property ki_fp_filters "TO-???* *_Diode_* *SingleDiode* D_*")
 		(sheetname "/")
-		(sheetfile "esphome-pc-power-dongle.kicad_sch")
+		(sheetfile "boop.kicad_sch")
 		(units
 			(unit
@@
 		(property ki_fp_filters "Connector*:*_1x??_*")
 		(sheetname "/")
-		(sheetfile "esphome-pc-power-dongle.kicad_sch")
+		(sheetfile "boop.kicad_sch")
 		(units
 			(unit
@@
 		(property ki_fp_filters "TO-???* *_Diode_* *SingleDiode* D_*")
 		(sheetname "/")
-		(sheetfile "esphome-pc-power-dongle.kicad_sch")
+		(sheetfile "boop.kicad_sch")
 		(units
 			(unit
@@
 			)
 		)
-		(property "Value" "G6K-2F-Y-TR DC5"
+		(property "Value" "G6K-2F-Y-TR DC4.5"
 			(at -0.04 6.3 90)
 			(layer "F.Fab")
@@
 			)
 		)
-		(property "LCSC" "C47190"
+		(property "LCSC" "C397193"
 			(at 0 0 90)
 			(unlocked yes)
@@
 		(property ki_fp_filters "Relay*DPDT*Omron*G6K?2*")
 		(sheetname "/")
-		(sheetfile "esphome-pc-power-dongle.kicad_sch")
+		(sheetfile "boop.kicad_sch")
 		(units
 			(unit
@@
 		(property ki_fp_filters "DIP*W7.62mm*")
 		(sheetname "/")
-		(sheetfile "esphome-pc-power-dongle.kicad_sch")
+		(sheetfile "boop.kicad_sch")
 		(units
 			(unit
@@
 		(layer "Edge.Cuts")
 	)
-	(gr_text "MB"
-		(at 162 117.3 0)
-		(layer "F.SilkS")
-		(effects
-			(font
-				(size 1 1)
-				(thickness 0.15)
-			)
-		)
-	)
-	(gr_text "CASE"
-		(at 166 117.3 0)
-		(layer "F.SilkS")
-		(effects
-			(font
-				(size 1 1)
-				(thickness 0.15)
-			)
-		)
-	)
 	(gr_text "5V IN"
 		(at 108 85.8 0)
@@
 		)
 	)
+	(gr_text "MB"
+		(at 162 117.3 0)
+		(layer "F.SilkS")
+		(effects
+			(font
+				(size 1 1)
+				(thickness 0.15)
+			)
+		)
+	)
 	(gr_text "PWR LED"
 		(at 164 85.8 0)
@@
 		(layer "F.SilkS")
 		(effects
+			(font
+				(size 1 1)
+				(thickness 0.15)
+			)
+		)
+	)
+	(gr_text "CASE"
+		(at 166 117.3 0)
+		(layer "F.SilkS")
+		(effects
